File: KiCad/christmas.kicad_sch (KiCad schematic)
At the start: 8 parts, among them U1 ICM7555xP, U2 4021, U3 ICM7555xP

Commit message: minor fixes
Parts:
- removed R2: R, symbol Device:R
- removed RV1, RV2: R_Potentiometer, symbol Device:R_Potentiometer
- removed U1, U3: ICM7555xP, Package_DIP:DIP-8_W7.62mm, symbol Timer:ICM7555xP
- removed U2: 4021, symbol 4xxx:4021
- added BT1: Battery_Cell, symbol Device:Battery_Cell
- added C1: 100n, symbol Device:C
- added D2, D3, D4, D5, D6, D7, D8: LED, LED_THT:LED_D5.0mm, symbol Device:LED
- added J1, J2: Conn_01x03, Connector_PinHeader_2.54mm:PinHeader_1x03_P2.54mm_Vertical, symbol Connector_Generic:Conn_01x03
- added JP1, JP2: Jumper_3_Open, Connector_PinHeader_2.54mm:PinHeader_1x03_P2.54mm_Vertical, symbol Jumper:Jumper_3_Open
- added R3, R4, R5, R6, R7, R8, R9: R, Resistor_THT:R_Axial_DIN0207_L6.3mm_D2.5mm_P7.62mm_Horizontal, symbol Device:R
- added U4: 74HC595, symbol 74xx:74HC595
- R1: footprint (none) -> Resistor_THT:R_Axial_DIN0207_L6.3mm_D2.5mm_P7.62mm_Horizontal
Connections:
- net GND: now also D1.1 (K), BT1.2 (-), C1.1, D2.1 (K), D3.1 (K), D4.1 (K), D5.1 (K), D6.1 (K), D7.1 (K), D8.1 (K), J1.3 (Pin_3), J2.3 (Pin_3), U4.13 (~{OE}), U4.8 (GND)
- net VCC: now also BT1.1 (+), C1.2, U4.16 (VCC); no longer R1.1
- net at D1.2 (A): now also R1.2
- new net: R7.1, U4.2 (QC)
- new net: D6.2 (A), R7.2
- new net: J1.1 (Pin_1), JP2.2 (C)
- new net: J1.2 (Pin_2), JP1.2 (C)
- new net: R1.1, U4.7 (QH)
- new net: R9.1, U4.15 (QA)
- new net: D8.2 (A), R9.2
- new net: D2.2 (A), R3.2
- new net: D5.2 (A), R6.2
- new net: J2.1 (Pin_1), JP2.3 (B), U4.14 (SER)
- new net: J2.2 (Pin_2), JP1.3 (B), U4.11 (SRCLK)
- new net: R4.1, U4.5 (QF)
- new net: D3.2 (A), R4.2
- new net: R8.1, U4.1 (QB)
- new net: R6.1, U4.3 (QD)
- new net: R5.1, U4.4 (QE)
- new net: R3.1, U4.6 (QG)
- new net: D4.2 (A), R5.2
- new net: D7.2 (A), R8.2
- new net Timer/Out: JP2.1 (A)
- new net Timer1/Out: JP1.1 (A)
Other:
- added sheet Timer (555Timer.kicad_sch)
- added sheet Timer1 (555Timer.kicad_sch)
- note added: "Supply Voltage: 2 bis 6"
- note added: "Supply Voltage: 4.5 bis 16"
- note removed: "555 Timer"
- note removed: "Output"
- note removed: "Shifting Register"
- moved on the sheet: D1

Commit message: minor fixes
Parts:
- removed J1, J2: Conn_01x03, Connector_PinHeader_2.54mm:PinHeader_1x03_P2.54mm_Vertical, symbol Connector_Generic:Conn_01x03
- removed U4: 74HC595, symbol 74xx:74HC595
- added D9: D, symbol Device:D
- added J1, J2: Conn_01x04, Connector_Molex:Molex_KK-254_AE-6410-04A_1x04_P2.54mm_Vertical, symbol Connector_Generic:Conn_01x04
- added JP3: Jumper_3_Open, Connector_PinHeader_2.54mm:PinHeader_1x03_P2.54mm_Vertical, symbol Jumper:Jumper_3_Open
- added U2: 4015, Package_DIP:DIP-16_W10.16mm_LongPads, symbol 4xxx_IEEE:4015
- C1: footprint (none) -> Capacitor_THT:C_Disc_D5.0mm_W2.5mm_P5.00mm
Connections:
- net GND: now also J1.4 (Pin_4), J2.4 (Pin_4), U2.14 (MR), U2.6 (MR), U2.8 (Vss), U2.8 (Vss)
- net Timer/Out: now also JP1.3 (B); no longer JP2.1 (A)
- net Timer1/Out: now also JP2.3 (B); no longer JP1.1 (A)
- net VCC: now also D9.1 (K), J2.3 (Pin_3), U2.16 (Vdd), U2.16 (Vdd)
- net at R7.1: now also U2.3 (Q3)
- net at JP2.2 (C): now also JP3.1 (A), U2.1 (CP), U2.9 (CP)
- net at JP1.2 (C): now also J2.2 (Pin_2), U2.7 (D)
- net at R1.1: now also JP3.3 (B), U2.2 (Q4)
- net at R9.1: now also U2.5 (Q1)
- net at R4.1: now also U2.12 (Q2)
- net at R8.1: now also U2.4 (Q2)
- net at R6.1: now also U2.10 (Q4), U2.15 (D)
- net at R5.1: now also U2.13 (Q1)
- net at R3.1: now also U2.11 (Q3)
- new net: J2.1 (Pin_1), JP3.2 (C)
- new net: J1.1 (Pin_1), JP2.1 (A)
- new net: J1.2 (Pin_2), JP1.1 (A)
- new net: D9.2 (A), J1.3 (Pin_3)
Other:
- note removed: "Supply Voltage: 2 bis 6"
- note removed: "Supply Voltage: 4.5 bis 16"
- moved on the sheet: BT1, C1, D1, D2, D3, D4, D5, D6, D7, D8, JP1, JP2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

Commit message: added pictures
Parts:
- removed BT1: Battery_Cell, symbol Device:Battery_Cell
- added H1, H2: MountingHole, MountingHole:MountingHole_2.2mm_M2, symbol Mechanical:MountingHole
Changed lines of the file:
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@@
-    )
-  )
-  (symbol (lib_id "Device:Battery_Cell") (at 68.58 153.67 0) (unit 1)
-    (in_bom yes) (on_board yes) (dnp no) (fields_autoplaced)
-    (property "Reference" "BT1" (at 72.39 150.5585 0)
-      (effects (font (size 1.27 1.27)) (justify left))
-    )
-    (property "Value" "Battery_Cell" (at 72.39 153.0985 0)
-      (effects (font (size 1.27 1.27)) (justify left))
-    )
-    (property "Footprint" "" (at 68.58 152.146 90)
-      (effects (font (size 1.27 1.27)) hide)
-    )
-    (property "Datasheet" "~" (at 68.58 152.146 90)
-      (effects (font (size 1.27 1.27)) hide)
-    )
-    (pin "1")
-    (pin "2")
-    (instances
-      (project "christmas"
-        (path "/3a264a14-3d89-40c1-a547-b76d7ed1f045"
-          (reference "BT1") (unit 1)
-        )
-      )
     )
   )
@@
     )
   )
+  (symbol (lib_id "Mechanical:MountingHole") (at 205.74 35.56 0) (unit 1)
+    (in_bom yes) (on_board yes) (dnp no) (fields_autoplaced)
+    (property "Reference" "H1" (at 208.28 34.29 0)
+      (effects (font (size 1.27 1.27)) (justify left))
+    )
+    (property "Value" "MountingHole" (at 208.28 36.83 0)
+      (effects (font (size 1.27 1.27)) (justify left))
+    )
+    (property "Footprint" "MountingHole:MountingHole_2.2mm_M2" (at 205.74 35.56 0)
+      (effects (font (size 1.27 1.27)) hide)
+    )
+    (property "Datasheet" "~" (at 205.74 35.56 0)
+      (effects (font (size 1.27 1.27)) hide)
+    )
+    (instances
+      (project "christmas"
+        (path "/3a264a14-3d89-40c1-a547-b76d7ed1f045"
+          (reference "H1") (unit 1)
+        )
+      )
+    )
+  )
   (symbol (lib_id "power:VCC") (at 152.4 63.5 0) (unit 1)
     (in_bom yes) (on_board yes) (dnp no)
@@
         (path "/3a264a14-3d89-40c1-a547-b76d7ed1f045/dd786dbd-2c93-405b-9b24-ff8effce1a4d"
           (reference "#PWR012") (unit 1)
-        )
-      )
-    )
-  )
-  (symbol (lib_id "power:VCC") (at 68.58 148.59 0) (unit 1)
-    (in_bom yes) (on_board yes) (dnp no)
-    (property "Reference" "#PWR029" (at 68.58 152.4 0)
-      (effects (font (size 1.27 1.27)) hide)
-    )
-    (property "Value" "VCC" (at 68.58 144.78 0)
-      (effects (font (size 1.27 1.27)))
-    )
-    (property "Footprint" "" (at 68.58 148.59 0)
-      (effects (font (size 1.27 1.27)) hide)
-    )
-    (property "Datasheet" "" (at 68.58 148.59 0)
-      (effects (font (size 1.27 1.27)) hide)
-    )
-    (pin "1")
-    (instances
-      (project "christmas"
-        (path "/3a264a14-3d89-40c1-a547-b76d7ed1f045"
-          (reference "#PWR029") (unit 1)
         )
       )
@@
     )
   )
-  (symbol (lib_id "power:GND") (at 68.58 156.21 0) (unit 1)
-    (in_bom yes) (on_board yes) (dnp no) (fields_autoplaced)
-    (property "Reference" "#PWR028" (at 68.58 162.56 0)
-      (effects (font (size 1.27 1.27)) hide)
-    )
-    (property "Value" "GND" (at 68.58 161.29 0)
-      (effects (font (size 1.27 1.27)))
-    )
-    (property "Footprint" "" (at 68.58 156.21 0)
-      (effects (font (size 1.27 1.27)) hide)
-    )
-    (property "Datasheet" "" (at 68.58 156.21 0)
-      (effects (font (size 1.27 1.27)) hide)
-    )
-    (pin "1")
-    (instances
-      (project "christmas"
-        (path "/3a264a14-3d89-40c1-a547-b76d7ed1f045"
-          (reference "#PWR028") (unit 1)
-        )
-        (path "/3a264a14-3d89-40c1-a547-b76d7ed1f045/dd786dbd-2c93-405b-9b24-ff8effce1a4d"
-          (reference "#PWR012") (unit 1)
-        )
-      )
-    )
-  )
   (symbol (lib_id "Device:LED") (at 214.63 114.3 90) (unit 1)
     (in_bom yes) (on_board yes) (dnp no) (fields_autoplaced)
@@
         )
       )
+    )
+  )
+  (symbol (lib_id "Mechanical:MountingHole") (at 205.74 40.64 0) (unit 1)
+    (in_bom yes) (on_board yes) (dnp no) (fields_autoplaced)
+    (property "Reference" "H2" (at 208.28 39.37 0)
+      (effects (font (size 1.27 1.27)) (justify left))
+    )
+    (property "Value" "MountingHole" (at 208.28 41.91 0)
+      (effects (font (size 1.27 1.27)) (justify left))
+    )
+    (property "Footprint" "MountingHole:MountingHole_2.2mm_M2" (at 205.74 40.64 0)
+      (effects (font (size 1.27 1.27)) hide)
+    )
+    (property "Datasheet" "~" (at 205.74 40.64 0)
+      (effects (font (size 1.27 1.27)) hide)
+    )
+    (instances
+      (project "christmas"
+        (path "/3a264a14-3d89-40c1-a547-b76d7ed1f045"
+          (reference "H2") (unit 1)
+        )
+      )
