File: KiCad/christmas.kicad_sch (KiCad schematic)
At the start: 26 parts, among them J1 Conn_01x04, J2 Conn_01x04, U2 4015

Commit message: minor fixchanges
Parts:
- added J3: Conn_01x02, Connector_PinHeader_2.54mm:PinHeader_1x02_P2.54mm_Vertical, symbol Connector_Generic:Conn_01x02
- D9: footprint (none) -> Diode_THT:D_5W_P5.08mm_Vertical_AnodeUp
- J1: footprint Connector_Molex:Molex_KK-254_AE-6410-04A_1x04_P2.54mm_Vertical -> Connector_JST:JST_XH_S4B-XH-A_1x04_P2.50mm_Horizontal
- J2: footprint Connector_Molex:Molex_KK-254_AE-6410-04A_1x04_P2.54mm_Vertical -> Connector_JST:JST_XH_S4B-XH-A-1_1x04_P2.50mm_Horizontal
Connections:
- net GND: now also J3.1 (Pin_1)
- net VCC: now also J3.2 (Pin_2)
Other:
- moved on the sheet: H1, H2
Changed lines of the file:
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@@
   (junction (at 149.86 123.19) (diameter 0) (color 0 0 0 0)
   )
+  (wire (pts (xy 68.58 161.29) (xy 71.12 161.29))
+    (stroke (width 0) (type default))
+  )
   (wire (pts (xy 85.09 96.52) (xy 85.09 93.98))
     (stroke (width 0) (type default))
@@
     (stroke (width 0) (type default))
   )
+  (wire (pts (xy 71.12 156.21) (xy 71.12 158.75))
+    (stroke (width 0) (type default))
+  )
   (wire (pts (xy 97.79 66.04) (xy 97.79 78.74))
     (stroke (width 0) (type default))
@@
     (stroke (width 0) (type default))
   )
+  (wire (pts (xy 71.12 161.29) (xy 71.12 163.83))
+    (stroke (width 0) (type default))
+  )
   (wire (pts (xy 214.63 125.73) (xy 214.63 85.09))
     (stroke (width 0) (type default))
@@
     (stroke (width 0) (type default))
   )
+  (wire (pts (xy 71.12 158.75) (xy 68.58 158.75))
+    (stroke (width 0) (type default))
+  )
   (wire (pts (xy 149.86 137.16) (xy 113.03 137.16))
     (stroke (width 0) (type default))
@@
     )
   )
-  (symbol (lib_id "Mechanical:MountingHole") (at 76.2 137.16 0) (unit 1)
-    (in_bom yes) (on_board yes) (dnp no) (fields_autoplaced)
-    (property "Reference" "H1" (at 78.74 135.89 0)
-      (effects (font (size 1.27 1.27)) (justify left))
-    )
-    (property "Value" "MountingHole" (at 78.74 138.43 0)
-      (effects (font (size 1.27 1.27)) (justify left))
-    )
-    (property "Footprint" "MountingHole:MountingHole_2.2mm_M2" (at 76.2 137.16 0)
-      (effects (font (size 1.27 1.27)) hide)
-    )
-    (property "Datasheet" "~" (at 76.2 137.16 0)
+  (symbol (lib_id "Mechanical:MountingHole") (at 72.39 130.81 0) (unit 1)
+    (in_bom yes) (on_board yes) (dnp no) (fields_autoplaced)
+    (property "Reference" "H1" (at 74.93 129.54 0)
+      (effects (font (size 1.27 1.27)) (justify left))
+    )
+    (property "Value" "MountingHole" (at 74.93 132.08 0)
+      (effects (font (size 1.27 1.27)) (justify left))
+    )
+    (property "Footprint" "MountingHole:MountingHole_2.2mm_M2" (at 72.39 130.81 0)
+      (effects (font (size 1.27 1.27)) hide)
+    )
+    (property "Datasheet" "~" (at 72.39 130.81 0)
       (effects (font (size 1.27 1.27)) hide)
     )
@@
     )
   )
+  (symbol (lib_id "power:GND") (at 71.12 163.83 0) (unit 1)
+    (in_bom yes) (on_board yes) (dnp no) (fields_autoplaced)
+    (property "Reference" "#PWR028" (at 71.12 170.18 0)
+      (effects (font (size 1.27 1.27)) hide)
+    )
+    (property "Value" "GND" (at 71.12 168.91 0)
+      (effects (font (size 1.27 1.27)))
+    )
+    (property "Footprint" "" (at 71.12 163.83 0)
+      (effects (font (size 1.27 1.27)) hide)
+    )
+    (property "Datasheet" "" (at 71.12 163.83 0)
+      (effects (font (size 1.27 1.27)) hide)
+    )
+    (pin "1")
+    (instances
+      (project "christmas"
+        (path "/3a264a14-3d89-40c1-a547-b76d7ed1f045"
+          (reference "#PWR028") (unit 1)
+        )
+        (path "/3a264a14-3d89-40c1-a547-b76d7ed1f045/dd786dbd-2c93-405b-9b24-ff8effce1a4d"
+          (reference "#PWR012") (unit 1)
+        )
+      )
+    )
+  )
   (symbol (lib_id "power:GND") (at 125.73 95.25 0) (unit 1)
     (in_bom yes) (on_board yes) (dnp no)
@@
       (effects (font (size 1.27 1.27)))
     )
-    (property "Footprint" "Connector_Molex:Molex_KK-254_AE-6410-04A_1x04_P2.54mm_Vertical" (at 63.5 60.96 0)
+    (property "Footprint" "Connector_JST:JST_XH_S4B-XH-A_1x04_P2.50mm_Horizontal" (at 63.5 60.96 0)
       (effects (font (size 1.27 1.27)) hide)
     )
@@
       (effects (font (size 1.27 1.27)))
     )
-    (property "Footprint" "Connector_Molex:Molex_KK-254_AE-6410-04A_1x04_P2.54mm_Vertical" (at 125.73 60.96 0)
+    (property "Footprint" "Connector_JST:JST_XH_S4B-XH-A-1_1x04_P2.50mm_Horizontal" (at 125.73 60.96 0)
       (effects (font (size 1.27 1.27)) hide)
     )
@@
     )
   )
+  (symbol (lib_id "power:VCC") (at 71.12 156.21 0) (unit 1)
+    (in_bom yes) (on_board yes) (dnp no)
+    (property "Reference" "#PWR04" (at 71.12 160.02 0)
+      (effects (font (size 1.27 1.27)) hide)
+    )
+    (property "Value" "VCC" (at 71.12 152.4 0)
+      (effects (font (size 1.27 1.27)))
+    )
+    (property "Footprint" "" (at 71.12 156.21 0)
+      (effects (font (size 1.27 1.27)) hide)
+    )
+    (property "Datasheet" "" (at 71.12 156.21 0)
+      (effects (font (size 1.27 1.27)) hide)
+    )
+    (pin "1")
+    (instances
+      (project "christmas"
+        (path "/3a264a14-3d89-40c1-a547-b76d7ed1f045"
+          (reference "#PWR04") (unit 1)
+        )
+        (path "/3a264a14-3d89-40c1-a547-b76d7ed1f045/dd786dbd-2c93-405b-9b24-ff8effce1a4d"
+          (reference "#PWR011") (unit 1)
+        )
+      )
+    )
+  )
+  (symbol (lib_id "Connector_Generic:Conn_01x02") (at 63.5 161.29 180) (unit 1)
+    (in_bom yes) (on_board yes) (dnp no) (fields_autoplaced)
+    (property "Reference" "J3" (at 63.5 152.4 0)
+      (effects (font (size 1.27 1.27)))
+    )
+    (property "Value" "Conn_01x02" (at 63.5 154.94 0)
+      (effects (font (size 1.27 1.27)))
+    )
+    (property "Footprint" "Connector_PinHeader_2.54mm:PinHeader_1x02_P2.54mm_Vertical" (at 63.5 161.29 0)
+      (effects (font (size 1.27 1.27)) hide)
+    )
+    (property "Datasheet" "~" (at 63.5 161.29 0)
+      (effects (font (size 1.27 1.27)) hide)
+    )
+    (pin "1")
+    (pin "2")
+    (instances
+      (project "christmas"
+        (path "/3a264a14-3d89-40c1-a547-b76d7ed1f045"
+          (reference "J3") (unit 1)
+        )
+      )
+    )
+  )
   (symbol (lib_id "power:GND") (at 154.94 140.97 0) (unit 1)
     (in_bom yes) (on_board yes) (dnp no)
@@
       (effects (font (size 1.27 1.27)) (justify left))
     )
-    (property "Footprint" "" (at 71.12 52.07 0)
+    (property "Footprint" "Diode_THT:D_5W_P5.08mm_Vertical_AnodeUp" (at 71.12 52.07 0)
       (effects (font (size 1.27 1.27)) hide)
     )
@@
     )
   )
-  (symbol (lib_id "Mechanical:MountingHole") (at 76.2 142.24 0) (unit 1)
-    (in_bom yes) (on_board yes) (dnp no) (fields_autoplaced)
-    (property "Reference" "H2" (at 78.74 140.97 0)
-      (effects (font (size 1.27 1.27)) (justify left))
-    )
-    (property "Value" "MountingHole" (at 78.74 143.51 0)
-      (effects (font (size 1.27 1.27)) (justify left))
-    )
-    (property "Footprint" "MountingHole:MountingHole_2.2mm_M2" (at 76.2 142.24 0)
-      (effects (font (size 1.27 1.27)) hide)
-    )
-    (property "Datasheet" "~" (at 76.2 142.24 0)
-      (effects (font (size 1.27 1.27)) hide)
-    )
+  (symbol (lib_id "Mechanical:MountingHole") (at 72.39 135.89 0) (unit 1)
+    (in_bom yes) (on_board yes) (dnp no) (fields_autoplaced)
+    (property "Reference" "H2" (at 74.93 134.62 0)
+      (effects (font (size 1.27 1.27)) (justify left))
+    )
+    (property "Value" "MountingHole" (at 74.93 137.16 0)
+      (effects (font (size 1.27 1.27)) (justify left))
+    )
+    (property "Footprint" "MountingHole:MountingHole_2.2mm_M2" (at 72.39 135.89 0)
+      (effects (font (size 1.27 1.27)) hide)
+    )
+    (property "Datasheet" "~" (at 72.39 135.89 0)
+      (effects (font (size 1.27 1.27)) hide)
+    )

Commit message: major fixes
Parts:
- removed D9: D, Diode_THT:D_5W_P5.08mm_Vertical_AnodeUp, symbol Device:D
- J3: value Conn_01x02 -> Batery_9V
- R1, R3, R4, R5, R6, R7, R8, R9: value R -> 1.4k
Connections:
- net VCC: now also J1.3 (Pin_3)
- net at JP2.2 (C), U2.1 (CP), U2.9 (CP): now also J2.1 (Pin_1); no longer JP3.1 (A)
- net at JP3.2 (C): now also J2.2 (Pin_2); no longer J2.1 (Pin_1)
- net Clk: now reaches J1.1 (Pin_1), JP2.1 (A)
- net Data: now reaches J1.2 (Pin_2), JP1.1 (A)
- net at JP1.2 (C), U2.7 (D): now also JP3.1 (A); no longer J2.2 (Pin_2)
Other:
- moved on the sheet: C1, H1, H2, J1, J2, J3, JP1, JP2, JP3
