File: KiCad/christmas.kicad_pcb (KiCad board)
At the start: 2 copper layers, 81.3 x 81.3 mm, 35 parts, among them J1 Conn_01x04, J2 Conn_01x04, U1 NE555P, U2 4015, U3 NE555P

Commit message: added pictures
Parts:
- added H1: MountingHole, MountingHole:MountingHole_2.2mm_M2, F.Cu at (182.4, 96.5)
- added H2: MountingHole, MountingHole:MountingHole_2.2mm_M2, F.Cu at (182.4, 109.1)
Routing:
- net Net-(U2B-Q3): track 26.8 -> 27.5 mm
Changed lines of the file:
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@@
     )
+  )
+  (footprint "MountingHole:MountingHole_2.2mm_M2" (layer "F.Cu")
+    (at 182.4 96.52)
+    (descr "Mounting Hole 2.2mm, no annular, M2")
+    (tags "mounting hole 2.2mm no annular m2")
+    (property "Sheetfile" "christmas.kicad_sch")
+    (property "Sheetname" "")
+    (property "ki_description" "Mounting Hole without connection")
+    (property "ki_keywords" "mounting hole")
+    (attr exclude_from_pos_files)
+    (fp_text reference "H1" (at 0 -3.2) (layer "F.SilkS")
+        (effects (font (size 1 1) (thickness 0.15)))
+    )
+    (fp_text value "MountingHole" (at 0 3.2) (layer "F.Fab") hide
+        (effects (font (size 1 1) (thickness 0.15)))
+    )
+    (fp_text user "${REFERENCE}" (at 0 0) (layer "F.Fab") hide
+        (effects (font (size 1 1) (thickness 0.15)))
+    )
+    (fp_circle (center 0 0) (end 2.2 0)
+      (stroke (width 0.15) (type solid)) (fill none) (layer "Cmts.User"))
+    (fp_circle (center 0 0) (end 2.45 0)
+      (stroke (width 0.05) (type solid)) (fill none) (layer "F.CrtYd"))
+    (pad "" np_thru_hole circle (at 0 0) (size 2.2 2.2) (drill 2.2) (layers "*.Cu" "*.Mask"))
   )
   (footprint "LED_THT:LED_D5.0mm" (layer "F.Cu")
@@
       (rotate (xyz 0 0 0))
     )
+  )
+  (footprint "MountingHole:MountingHole_2.2mm_M2" (layer "F.Cu")
+    (at 182.4 109.1)
+    (descr "Mounting Hole 2.2mm, no annular, M2")
+    (tags "mounting hole 2.2mm no annular m2")
+    (property "Sheetfile" "christmas.kicad_sch")
+    (property "Sheetname" "")
+    (property "ki_description" "Mounting Hole without connection")
+    (property "ki_keywords" "mounting hole")
+    (attr exclude_from_pos_files)
+    (fp_text reference "H2" (at 0 -3.2) (layer "F.SilkS")
+        (effects (font (size 1 1) (thickness 0.15)))
+    )
+    (fp_text value "MountingHole" (at 0 3.2) (layer "F.Fab") hide
+        (effects (font (size 1 1) (thickness 0.15)))
+    )
+    (fp_text user "${REFERENCE}" (at 0 0) (layer "F.Fab") hide
+        (effects (font (size 1 1) (thickness 0.15)))
+    )
+    (fp_circle (center 0 0) (end 2.2 0)
+      (stroke (width 0.15) (type solid)) (fill none) (layer "Cmts.User"))
+    (fp_circle (center 0 0) (end 2.45 0)
+      (stroke (width 0.05) (type solid)) (fill none) (layer "F.CrtYd"))
+    (pad "" np_thru_hole circle (at 0 0) (size 2.2 2.2) (drill 2.2) (layers "*.Cu" "*.Mask"))
   )
   (footprint "Resistor_THT:R_Axial_DIN0207_L6.3mm_D2.5mm_P7.62mm_Horizontal" (layer "F.Cu")
@@
   (segment (start 174.248 98.04) (end 174.752 97.536) (width 0.6) (layer "F.Cu") (net 26))
   (segment (start 174.752 93.324892) (end 167.787108 86.36) (width 0.6) (layer "F.Cu") (net 26))
-  (segment (start 187.066048 93.399962) (end 187.066048 97.413952) (width 0.6) (layer "F.Cu") (net 27))
-  (segment (start 179.07 105.41) (end 167.64 105.41) (width 0.6) (layer "F.Cu") (net 27))
-  (segment (start 187.066048 97.413952) (end 179.07 105.41) (width 0.6) (layer "F.Cu") (net 27))
+  (segment (start 180.34 105.41) (end 167.64 105.41) (width 0.6) (layer "F.Cu") (net 27))
+  (segment (start 187.066048 93.399962) (end 187.066048 98.683952) (width 0.6) (layer "F.Cu") (net 27))
+  (segment (start 187.066048 98.683952) (end 180.34 105.41) (width 0.6) (layer "F.Cu") (net 27))
   (segment (start 165.1 111.125) (end 166.37 112.395) (width 0.6) (layer "F.Cu") (net 28))
   (segment (start 166.37 112.395) (end 174.625 112.395) (width 0.6) (layer "F.Cu") (net 28))
@@
   (segment (start 148.652892 116.84) (end 134.910019 130.582873) (width 0.6) (layer "B.Cu") (net 30))
   (segment (start 166.37 107.95) (end 157.48 116.84) (width 0.6) (layer "B.Cu") (net 30))
-  (segment (start 124.815995 103.886) (end 117.921976 110.780019) (width 0.6) (layer "B.Cu") (net 31))
-  (segment (start 151.13 104.14) (end 150.876 103.886) (width 0.6) (layer "B.Cu") (net 31))
-  (segment (start 157.48 97.79) (end 151.13 104.14) (width 0.6) (layer "B.Cu") (net 31))
-  (segment (start 150.876 103.886) (end 124.815995 103.886) (width 0.6) (layer "B.Cu") (net 31))
+  (segment (start 124.815995 103.886) (end 124.510998 104.190998) (width 0.6) (layer "B.Cu") (net 31))
+  (segment (start 149.479 103.886) (end 155.575 97.79) (width 0.6) (layer "B.Cu") (net 31))
+  (segment (start 124.510998 104.190998) (end 117.921976 110.780019) (width 0.6) (layer "B.Cu") (net 31))
+  (segment (start 124.815996 103.886) (end 149.479 103.886) (width 0.6) (layer "B.Cu") (net 31))
+  (segment (start 124.510998 104.190998) (end 124.815996 103.886) (width 0.6) (layer "B.Cu") (net 31))
+  (segment (start 155.575 97.79) (end 157.48 97.79) (width 0.6) (layer "B.Cu") (net 31))
   (segment (start 134.62 77.47) (end 127.979981 84.110019) (width 0.6) (layer "F.Cu") (net 32))
   (segment (start 127.979981 84.110019) (end 122.108024 84.110019) (width 0.6) (layer "F.Cu") (net 32))

Commit message: minor fixchanges
Parts:
- added D9: D, Diode_THT:D_5W_P5.08mm_Vertical_AnodeUp, F.Cu at (212.1, 116.2)
- added J3: Conn_01x02, Connector_PinHeader_2.54mm:PinHeader_1x02_P2.54mm_Vertical, F.Cu at (211.7, 121.3)
- J1: footprint Connector_Molex:Molex_KK-254_AE-6410-04A_1x04_P2.54mm_Vertical -> Connector_JST:JST_XH_S4B-XH-A_1x04_P2.50mm_Horizontal
- J2: footprint Connector_Molex:Molex_KK-254_AE-6410-04A_1x04_P2.54mm_Vertical -> Connector_JST:JST_XH_S4B-XH-A-1_1x04_P2.50mm_Horizontal

Commit message: major fixes
Parts:
- removed D9: D, Diode_THT:D_5W_P5.08mm_Vertical_AnodeUp
- J3: value Conn_01x02 -> Batery_9V
- R1, R3, R4, R5, R6, R7, R8, R9: value R -> 1.4k
- moved J3 48.5 mm to (177.9, 86.5), turned to 45 degrees
- moved J1 4.55 mm to (162.4, 84.6)
- moved J2 4.48 mm to (170.0, 118.6)
Connections:
- net Net-(J1-Pin_1) renamed /Clk
- net Net-(J1-Pin_2) renamed /Data
- J1 pad 3: Net-(D9-A) -> VCC
- JP1 pad 2: Net-(J2-Pin_2) -> Net-(JP1-C)
- JP2 pad 2: Net-(JP2-C) -> Net-(J2-Pin_1)
- JP3 pad 1: Net-(JP2-C) -> Net-(JP1-C)
- JP3 pad 2: Net-(J2-Pin_1) -> Net-(J2-Pin_2)
- U2 pad 1: Net-(JP2-C) -> Net-(J2-Pin_1)
- U2 pad 7: Net-(J2-Pin_2) -> Net-(JP1-C)
- U2 pad 9: Net-(JP2-C) -> Net-(J2-Pin_1)
Routing:
- net Net-(JP2-C): track 83.0 -> 0.00 mm, vias 3 -> 0
- net Net-(JP1-C): track 0.00 -> 72.0 mm
- net Net-(J2-Pin_1): track 33.0 -> 84.1 mm, vias 1 -> 5
- net Net-(J2-Pin_2): track 65.4 -> 24.9 mm, vias 1 -> 0
- net VCC: track 124.6 -> 142.8 mm
- net Net-(JP3-B): track 54.1 -> 47.1 mm
- net /Data: track 77.4 -> 70.6 mm
- net /Clk: track 45.7 -> 40.9 mm
- net Net-(U2B-Q1): track 37.9 -> 39.0 mm
- net Net-(U2A-Q4): track 58.4 -> 57.9 mm
