File: KiCad/christmas.kicad_pcb (KiCad board)
At the start: 2 copper layers, 81.3 x 81.3 mm, 42 parts, among them J1 Conn_01x04, J2 Conn_01x04, J3 Battery_9V, U1 NE555P, U2 4015, U3 NE555P

Commit message: switch Poti wiring, adjust to JLCPCB design rules
Connections:
- RV1 pad 1: Net-(R2-Pad1) -> Net-(U1-THR)
- RV1 pad 3: Net-(U1-THR) -> Net-(R2-Pad1)
- RV2 pad 1: Net-(R10-Pad1) -> Net-(U3-THR)
- RV2 pad 3: Net-(U3-THR) -> Net-(R10-Pad1)
Routing:
- net Net-(R10-Pad1): track 29.6 -> 20.0 mm
- net Net-(R2-Pad1): track 28.2 -> 25.0 mm
- net Net-(U2A-Q3): track 61.2 -> 63.7 mm
- net Net-(U1-THR): track 25.8 -> 28.3 mm
- net Net-(U2B-Q2): track 69.6 -> 70.2 mm
- net VCC: vias 1 -> 0
- net GND: vias 5 -> 6
Other:
- board text added: "Data"
- board text added: "J1: Data IN: Own Timer / Input J2: Clock IN: Own Timer / Input J3: Data OUT: Series / Parallel"
- board text removed: "J1: Data: Own Timer / IN J2: Clock: Own Timer / IN J3: Push OUT: Data Timer / Shiftregister out"
