File: KiCad/_autosave-christmas.kicad_sch (KiCad schematic)
At the start: 28 parts, among them J1 Conn_01x04, J2 Conn_01x04, J3 Battery_9V, U2 4015

Commit message: restructure components on board and implement ToDos from prototyping
Parts:
- U2: footprint Package_DIP:DIP-16_W10.16mm_LongPads -> Package_DIP:DIP-16_W7.62mm_LongPads
Changed lines of the file:
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@@
       (effects (font (size 1.27 1.27)) (justify left))
     )
-    (property "Footprint" "Package_DIP:DIP-16_W10.16mm_LongPads" (at 132.08 120.65 0)
+    (property "Footprint" "Package_DIP:DIP-16_W7.62mm_LongPads" (at 132.08 120.65 0)
       (effects (font (size 1.27 1.27)) hide)
     )
@@
       (effects (font (size 1.27 1.27)) (justify left))
     )
-    (property "Footprint" "Package_DIP:DIP-16_W10.16mm_LongPads" (at 132.08 87.63 0)
-      (effects (font (size 1.27 1.27)) hide)
-    )
+    (property "Footprint" "Package_DIP:DIP-16_W7.62mm_LongPads" (at 132.08 87.63 0)
+      (effects (font (size 1.27 1.27)) hide)
+    )
